Commit message: [nextage_description] Add IK targets

File: nextage_description/urdf/NextageOpen.urdf.xacro (robot description, xacro)
@@ -488,4 +488,16 @@
     <dynamics damping="0.2" friction="0" />
   </joint>
+  <link name="LARM_TARGET"/>
+  <joint name="LARM_TARGET_JOINT" type="fixed">
+    <parent link="LARM_JOINT5_Link"/>
+    <child link="LARM_TARGET"/>
+    <origin xyz="-0.1 0.0 0.0" rpy="0 ${pi / 2.0} 0"/>
+  </joint>
+  <link name="RARM_TARGET"/>
+  <joint name="RARM_TARGET_JOINT" type="fixed">
+    <parent link="RARM_JOINT5_Link"/>
+    <child link="RARM_TARGET"/>
+    <origin xyz="-0.1 0.0 0.0" rpy="0 ${pi / 2.0} 0"/>
+  </joint>
   <!-- Gazebo plugin for ROS Control -->
   <gazebo>
